File: PSG-PCB/PSG-PCB.kicad_pcb (KiCad board)
At the start: 2 copper layers, 149.9 x 66 mm, 30 parts, among them J1 Jack_3.5mm_CUI_SJ1-3523N_Hori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, K1 Relay_DPDT_CIT_J104D, Q1 TO-92_Inline

Commit message: Redesigned board volume control, added version check
Parts:
- removed the ? at (101.6, 29.2)
- removed the ? at (155.0, 29.2)
- added R3: Potentiometer_Bourns_PDB182-K_Horizontal, Potentiometer_THT:Potentiometer_Bourns_PDB182-K_Horizontal, F.Cu at (92.7, 30.5)
- R2 (x2): value 910K -> 150K
- moved PICO 7.62 mm to (54.6, 38.1)
Connections:
- PICO pad 1: (no net) -> Ground
- PICO pad 2: (no net) -> Ground
- PICO pad 4: (no net) -> Ground
- PICO pad 5: (no net) -> Ground
- PICO pad 6: (no net) -> Ground
- PICO pad 7: (no net) -> VDD
Routing:
- net Audio_Out_R: track 8.33 -> 66.1 mm
- net Ground: track 37.2 -> 93.1 mm
- net Audio_In_R_Amp: track 9.89 -> 64.6 mm
- net D6: track 330.4 -> 301.9 mm, vias 1 -> 2
- net D7: track 321.5 -> 296.1 mm
- net SCL: track 254.9 -> 272.3 mm
- net VDD: track 32.1 -> 47.8 mm, vias 0 -> 2
- net D4: track 352.5 -> 339.5 mm
- net D3: track 363.9 -> 351.7 mm
- net D5: track 342.9 -> 330.9 mm
- net D0: track 397.4 -> 405.0 mm
- net Stereo: track 38.5 -> 46.1 mm
- net SDA: track 34.3 -> 42.0 mm
- net D2: track 420.4 -> 428.1 mm
- net D1: track 407.3 -> 415.0 mm
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Other:
- board text added: "Programmable Sound Generator Board v1.2.2 - 2022-12-16 Made by JackMacWindows"
- board text removed: "POT-L"
- board text removed: "POT-R"
- board text removed: "Programmable Sound Generator Board v1.2.1 - 2022-11-04 Made by JackMacWindows"
